File: pcb/esp32-mini-dev-board.kicad_sch (KiCad schematic)
At the start: 0 parts

Commit message: feat(arch): add top-level block diagram sheet
Other:
- added sheet BLOCK DIAGRAM (block-diagram.kicad_sch)
- added sheet CIRCUIT DESIGN (circuit-design.kicad_sch)
- note added: "INDEX"
- company: (none) -> NELSON RODRIGUEZ (LENZSEG)
- title: (none) -> ESP32 MINI DEV BOARD
Changed lines of the file:
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@@
 	(generator_version "10.0")
 	(paper "A4")
+	(title_block
+		(title "ESP32 MINI DEV BOARD")
+		(date "2026-09-30")
+		(rev "1.0")
+		(company "NELSON RODRIGUEZ (LENZSEG)")
+		(comment 1 "INDEX")
+	)
+	(text "INDEX"
+		(exclude_from_sim no)
+		(at 40.894 34.798 0)
+		(effects
+			(font
+				(face "KiCad Font")
+				(size 6.35 6.35)
+				(thickness 1.27)
+				(bold yes)
+			)
+		)
+	)
+	(sheet
+		(at 27.178 46.482)
+		(size 66.802 3.81)
+		(exclude_from_sim yes)
+		(in_bom no)
+		(on_board no)
+		(dnp no)
+		(fields_autoplaced yes)
+		(stroke
+			(width 0.254)
+			(type solid)
+		)
+		(fill
+			(color 0 0 0 0)
+		)
+		(property "Sheetname" "BLOCK DIAGRAM"
+			(at 27.178 45.7196 0)
+			(show_name no)
+			(do_not_autoplace no)
+			(effects
+				(font
+					(size 1.27 1.27)
+					(thickness 0.254)
+					(bold yes)
+				)
+				(justify left bottom)
+			)
+		)
+		(property "Sheetfile" "block-diagram.kicad_sch"
+			(at 27.178 50.9274 0)
+			(show_name no)
+			(do_not_autoplace no)
+			(effects
+				(font
+					(size 1.27 1.27)
+				)
+				(justify left top)
+			)
+		)
+		(instances
+			(project "esp32-mini-dev-board"
+				(path "/fce4255d-220c-4173-a7af-d7c1fd356d20"
+					(page "2")
+				)
+			)
+		)
+	)
+	(sheet
+		(at 26.67 62.23)
+		(size 67.31 3.81)
+		(exclude_from_sim no)
+		(in_bom yes)
+		(on_board yes)
+		(dnp no)
+		(fields_autoplaced yes)
+		(stroke
+			(width 0.254)
+			(type solid)
+		)
+		(fill
+			(color 0 0 0 0)
+		)
+		(property "Sheetname" "CIRCUIT DESIGN"
+			(at 26.67 61.4676 0)
+			(show_name no)
+			(do_not_autoplace no)
+			(effects
+				(font
+					(size 1.27 1.27)
+					(thickness 0.254)
+					(bold yes)
+				)
+				(justify left bottom)
+			)
+		)
+		(property "Sheetfile" "circuit-design.kicad_sch"
+			(at 26.67 66.6754 0)
+			(show_name no)
+			(do_not_autoplace no)
+			(effects
+				(font
+					(size 1.27 1.27)
+				)
+				(justify left top)
+			)
+		)
+		(instances
+			(project "esp32-mini-dev-board"
+				(path "/fce4255d-220c-4173-a7af-d7c1fd356d20"
+					(page "3")
+				)
+			)
+		)
+	)
 	(sheet_instances
 		(path "/"

Commit message: feat(lay): finish routing and copper pouring
Changed lines of the file:
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@@
 	(sheet
 		(at 27.178 46.482)
-		(size 66.802 3.81)
+		(size 66.802 10.16)
 		(exclude_from_sim yes)
 		(in_bom no)
@@
 		)
 		(property "Sheetfile" "block-diagram.kicad_sch"
-			(at 27.178 50.9274 0)
+			(at 27.178 57.2774 0)
 			(show_name no)
 			(do_not_autoplace no)
@@
 	)
 	(sheet
-		(at 26.67 62.23)
-		(size 67.31 3.81)
+		(at 27.432 67.31)
+		(size 67.31 9.652)
 		(exclude_from_sim no)
 		(in_bom yes)
@@
 		)
 		(property "Sheetname" "CIRCUIT DESIGN"
-			(at 26.67 61.4676 0)
+			(at 27.432 66.5476 0)
 			(show_name no)
 			(do_not_autoplace no)
@@
 		)
 		(property "Sheetfile" "circuit-design.kicad_sch"
-			(at 26.67 66.6754 0)
+			(at 27.432 77.5974 0)
 			(show_name no)
 			(do_not_autoplace no)
