File: pcb/esp32-mini-dev-board.kicad_pcb (KiCad board)
At the start: 4 copper layers, 30.4 x 37.8 mm, 32 parts, among them J1 USB_C_Receptacle_USB2.0_16P, J2 Conn_01x08_Pin, J3 Conn_01x08_Pin, U1 USBLC6-2SC6, U2 AP2112K-3.3, U3 ESP32-C3-WROOM-02, Y1 Crystal

Commit message: fix(lay): make several changes to pass JLCDFM tool check
- Copper zones were resize.
- Vias were shifter to avoid silkscreen graphical objects and text interference.
- Keep out zones were added to remove JLCDFM bug in soldermask expansion rule.
- Headers were moved away headers from ESP32-C3 module to pass tht-smt rule.
Parts:
- moved J2 0.40 mm to (149.6, 100.0)
- moved J3 0.40 mm to (176.4, 100.0)
Other:
- rule pad_to_mask_clearance: 0 -> 0.02
