File: src/esp32-mini-dev-board.kicad_pcb (KiCad board)
At the start: 4 copper layers, 30.4 x 37.8 mm, 32 parts, among them J1 USB_C_Receptacle_USB2.0_16P, J2 Conn_01x08_Pin, J3 Conn_01x08_Pin, U1 USBLC6-2SC6, U2 AP2112K-3.3, U3 ESP32-C3-WROOM-02, Y1 Crystal

Commit message: refactor(sch/usb): replace circuit protection devices symbols with own database symbols
Parts:
- removed the R6 at (167.5, 99.0)
- removed the R8 at (167.5, 100.5)
- added G***: LOGO, LZ Logos:lz-logo-3x3, F.Cu at (168.3, 114.2)
- C1, C11, C3: value C -> 4.7uF
- C10: value 100n -> C
- C2: value 4u7 -> 4.7uF; footprint Capacitor_SMD:C_0603_1608Metric -> #LZ_Capacitor_SMD:C_0603_1608Metric
- C4, C6, C8, C9: value 4u7 -> 4.7uF
- R1, R2: value 5k1 -> R
- R5: value 0R -> R
- Y1: value Crystal -> 32.768kHz
- moved R6 1.57 mm to (166.2, 101.0), turned to 0 degrees
- moved Y1 0.10 mm to (163.2, 99.8)
- moved C9 0.06 mm to (155.1, 100.5)
- renumbered R7 to R6, R9 to R7, R10 to R8, R11 to R9, RESET to SW1, BOOT to SW2
Connections:
- C5 pad 1: Net-(C5-Pad1) -> /CIRCUIT DESIGN/XTAL_32K_P
- R6 pad 1: Net-(C5-Pad1) -> Net-(C7-Pad1)
- R6 pad 2: Net-(C7-Pad1) -> /CIRCUIT DESIGN/XTAL_32K_N
- Y1 pad 1: Net-(C5-Pad1) -> /CIRCUIT DESIGN/XTAL_32K_P
Routing:
- net /CIRCUIT DESIGN/XTAL_32K_P: track 3.75 -> 10.7 mm
- net Net-(C5-Pad1): track 5.85 -> 0.00 mm
- net Net-(C7-Pad1): track 5.89 -> 4.23 mm
- net /CIRCUIT DESIGN/XTAL_32K_N: track 3.76 -> 5.32 mm
Other:
- board size 30.4 x 37.8 mm -> 30.4 x 38.1 mm
- board text added: "RST"
- board text removed: "LENZSEG"

Commit message: feat(sch): add MPN for RPUs and R filter
Parts:
- removed the G*** at (168.3, 114.2)
- added G***: LOGO, #LZ_Logos:lz-logo-3x3, F.Cu at (168.1, 113.9)
